File: usb_device.kicad_sch (KiCad schematic)
At the start: 1 part, among them J3 USB_C_Receptacle_USB2.0_16P

Commit message: More USB schematic work
Parts:
- added D2, D3, D4: LESD5D5.0CT1G, Diode_SMD:D_SOD-523, symbol Device:D_TVS_Small_Filled
- added R30, R31: 5.1K(1%), Resistor_SMD:R_0402_1005Metric, symbol Device:R_Small
Connections:
- net GND: now also D2.1 (A1), D3.1 (A1), D4.1 (A1), R30.1, R31.1
- net USB+: now also D2.2 (A2)
- net USB-: now also D3.2 (A2)
- net VBUS: now also D4.2 (A2)
- net at J3.A5 (CC1): now also R30.2
- net at J3.B5 (CC2): now also R31.2

Commit message: Getting close. Fault circuit left
Parts:
- J3: footprint (none) -> Adafruit:USB_C_Receptacle_HRO_TYPE-C-31-M-31
Connections:
- net VBUS renamed USB_5V
Other:
- removed sheet USBDiode
