File: faultcheck.kicad_sch (KiCad schematic)
At the start: 3 parts, among them U11 74AHC1G08, U12 74AUC1G74, U5 TLV7031DBV

Commit message: where I'm at. fault not needed
Parts:
- added R71: 10k, Resistor_SMD:R_0402_1005Metric, symbol Device:R_Small
- added R72: 30k, Resistor_SMD:R_0402_1005Metric, symbol Device:R_Small
- U11: footprint (none) -> Package_TO_SOT_SMD:SOT-23-5
- U12: footprint (none) -> Package_SO:VSSOP-8_2.3x2mm_P0.5mm
Connections:
- net +3.3V: now also U12.7 (~{PRE})
- net +5V: now also R71.1
- net GND: now also R72.2
- net at U5.3 (+): now also R71.2, R72.1
Other:
- note added: "3.75V or so"
