File: p4hil.kicad_pcb (KiCad board)
At the start: 4 copper layers, 66 x 53.3 mm, 62 parts, among them J10 Conn_01x22, J11 Conn_01x22, J12 Conn_01x22, J2 Conn_01x08, J4 Conn_01x10, J5 Conn_01x22, J6 Conn_01x22, J7 Conn_01x22, J9 Conn_01x06, U1 W25Q128JVS, U3 TLV62569DBV, Y1 40MHz(+-10 ppm) C501798

Commit message: More schematic work. Mostly on Ethernet
Parts:
- removed C40: 0.1uF, Capacitor_SMD:C_0402_1005Metric
- removed C41: 10nF, Capacitor_SMD:C_0402_1005Metric
- removed C42: 4.7uF, Capacitor_SMD:C_0402_1005Metric
- removed R28: 10k, Resistor_SMD:R_0402_1005Metric
- removed R39: 0, Resistor_SMD:R_0402_1005Metric
- added REF**: Converter_DCDC_Silvertel_Ag54xx, Converter_DCDC:Converter_DCDC_Silvertel_Ag54xx, F.Cu at (117.0, 69.1)
- C1, C10, C15, C17, C19, C22, C3, C4, C5, R5, R6, R7: moved to B.Cu
- C12, C14, C21, C25, C28, REF**: moved to F.Cu
- moved C11 338.5 mm to (133.1, 81.2), turned to 180 degrees
- moved C20 334.3 mm to (138.8, 87.7), turned to 90 degrees
- moved U3 334.0 mm to (150.5, 88.2), turned to 0 degrees
- moved U1 334.0 mm to (131.2, 81.0), turned to -90 degrees
- moved C24 333.6 mm to (143.2, 85.8), turned to 180 degrees
- moved C28 332.5 mm to (144.2, 91.5), turned to -90 degrees
- moved C3 326.7 mm to (141.6, 80.1), turned to 90 degrees
- moved C2 326.5 mm to (138.0, 80.7), turned to -90 degrees
- moved C8 325.3 mm to (146.9, 79.3), turned to 90 degrees
- moved C14 321.1 mm to (151.8, 84.4), turned to 180 degrees
- moved C1 320.4 mm to (143.2, 79.6), turned to 90 degrees
- moved C31 266.0 mm to (139.7, 91.8), turned to -90 degrees
- moved C13 264.1 mm to (133.1, 82.2), turned to 180 degrees
- moved C26 261.9 mm to (136.7, 91.4), turned to -90 degrees
- moved C32 261.4 mm to (143.4, 88.1)
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Connections:
- net /P4/GPIO24/ADC/USB_JTAG_DM renamed /USB_SERIAL-
- net /P4/GPIO25/ADC/USB_JTAG_DP renamed /USB_SERIAL+
- net /P4/GPIO28 renamed /RMII_CRSDV
- net /P4/GPIO29 renamed /RMII_RXD0
- net /P4/GPIO30 renamed /RMII_RXD1
- net /P4/GPIO31 renamed /RMII_RXER
- net /P4/GPIO32 renamed /RMII_CLK
- net /P4/GPIO33 renamed /RMII_TXEN
- net /P4/GPIO34 renamed /RMII_TXD0
- net /P4/GPIO35_BOOT_PULLUP renamed /RMII_TXD1
- net /P4/GPIO36_PULLUP renamed /RMII_TXER
- net /P4/HS_USB_D+ renamed /USB_HOST+
- net /P4/HS_USB_D- renamed /USB_HOST-
Routing:
- net /P4/VDD_HP: track 0.00 -> 58.1 mm, vias 0 -> 9
- net /Minimal P4 V3/VDD_HP: track 58.1 -> 0.00 mm, vias 9 -> 0
- net (no net): track 37.6 -> 0.00 mm, vias 3 -> 0
- net Net-(J10-Pin_15): track 0.00 -> 17.3 mm, vias 1 -> 0
- net /P4/FB_DCDC: track 0.00 -> 16.5 mm, vias 0 -> 2
- net /Minimal P4 V3/VDD_FLASH: track 9.81 -> 0.00 mm, vias 1 -> 0
- net /P4/FLASH_D: track 9.24 -> 0.00 mm
- net /P4/VDD_FLASH: track 0.62 -> 9.81 mm, vias 0 -> 1
- net /P4/FLASH_CK: track 8.05 -> 0.00 mm
- net Net-(J10-Pin_18): track 0.00 -> 7.15 mm
- net /P4/FLASH_Q: track 7.15 -> 0.00 mm
- net /Minimal P4 V3/FLASH_CS: track 5.00 -> 0.00 mm, vias 2 -> 0
- net /P4/FLASH_CS: track 0.00 -> 5.00 mm, vias 0 -> 2
- net /P4/EN_DCDC: track 0.00 -> 4.60 mm
- net Net-(C14-Pad1): track 0.00 -> 4.29 mm
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
Commit message: More USB schematic work
Parts:
- added REF**: Converter_DCDC_Silvertel_Ag99xxLP_THT, Converter_DCDC:Converter_DCDC_Silvertel_Ag99xxLP_THT, F.Cu at (171.6, 96.4)
- moved REF** 71.4 mm to (167.8, 18.9), turned to -90 degrees
- moved REF** 35.2 mm to (186.2, 66.5)
- moved REF** 2.72 mm to (109.0, 79.7)
- moved REF** 1.73 mm to (173.0, 87.2)
Other:
- board size 66 x 53.3 mm -> 81.3 x 50.8 mm

Commit message: Getting close. Fault circuit left
Parts:
- removed REF**: RJ45_Hanrun_HR911105A_Horizontal, Connector_RJ:RJ45_Hanrun_HR911105A_Horizontal
- removed REF**: USB_A_CUI_UJ2-ADH-TH_Horizontal_Stacked, Connector_USB:USB_A_CUI_UJ2-ADH-TH_Horizontal_Stacked
- removed REF**: Converter_DCDC_Silvertel_Ag99xxLP_THT, Converter_DCDC:Converter_DCDC_Silvertel_Ag99xxLP_THT
- removed REF**: USB_C_Receptacle_HRO_TYPE-C-31-M-12, Connector_USB:USB_C_Receptacle_HRO_TYPE-C-31-M-12
- removed REF**: Converter_DCDC_Silvertel_Ag54xx, Converter_DCDC:Converter_DCDC_Silvertel_Ag54xx
- added ACTIVE1: LED_Small, LED_SMD:LED_0603_1608Metric, F.Cu at (105.4, 94.8)
- added C35: 100nF, Capacitor_SMD:C_0402_1005Metric, F.Cu at (171.5, 51.4)
- added C36: 10uF, Capacitor_SMD:C_0603_1608Metric, F.Cu at (169.2, 65.6)
- added C37: 10uF, Capacitor_SMD:C_0603_1608Metric, F.Cu at (169.2, 68.1)
- added C38: 100nF, Capacitor_SMD:C_0402_1005Metric, F.Cu at (171.5, 53.3)
- added C39: 10uF, Capacitor_SMD:C_0603_1608Metric, F.Cu at (169.2, 70.6)
- added C40: 100nF, Capacitor_SMD:C_0402_1005Metric, F.Cu at (171.5, 55.3)
- added C41: 18pF, Capacitor_SMD:C_0402_1005Metric, F.Cu at (171.5, 57.3)
- added C42: 18pF, Capacitor_SMD:C_0402_1005Metric, F.Cu at (171.5, 59.2)
- added C43: 100nF, Capacitor_SMD:C_0402_1005Metric, B.Cu at (176.1, 83.5)
- added C46: 10uF, Capacitor_SMD:C_0603_1608Metric, F.Cu at (116.3, 88.6)
- added C47: 10uF, Capacitor_SMD:C_0603_1608Metric, F.Cu at (116.3, 91.1)
- added C48: 100nF, Capacitor_SMD:C_0402_1005Metric, F.Cu at (119.4, 90.0)
- added C49: 100nF, Capacitor_SMD:C_0402_1005Metric, F.Cu at (135.5, 64.8)
- added C50: 10uF, Capacitor_SMD:C_0603_1608Metric, F.Cu at (116.3, 115.3)
- added C51: 10uF, Capacitor_SMD:C_0603_1608Metric, F.Cu at (116.3, 117.8)
- added C52: 10uF, Capacitor_SMD:C_0603_1608Metric, F.Cu at (116.3, 120.3)
- added C53: 10uF, Capacitor_SMD:C_0603_1608Metric, F.Cu at (116.3, 122.8)
- added C54: 0.1uF, Capacitor_SMD:C_0402_1005Metric, F.Cu at (206.0, 132.7)
- added C55: 10uF, Capacitor_SMD:C_0603_1608Metric, F.Cu at (159.0, 135.3)
- added C56: 22pF, Capacitor_SMD:C_0402_1005Metric, F.Cu at (143.6, 137.5)
- added C57: 10uF, Capacitor_SMD:C_0603_1608Metric, F.Cu at (159.0, 137.8)
- added D1: WS2812B, LED_SMD:LED_WS2812B_PLCC4_5.0x5.0mm_P3.2mm, F.Cu at (205.8, 128.4)
- added D2: LESD5D5.0CT1G, Diode_SMD:D_SOD-523, F.Cu at (199.4, 84.2)
- added D3: LESD5D5.0CT1G, Diode_SMD:D_SOD-523, F.Cu at (201.8, 84.2)
- added D4: LESD5D5.0CT1G, Diode_SMD:D_SOD-523, F.Cu at (204.3, 84.2)
- added D8: GREEN LED, Diode_SMD:D_0805_2012Metric, F.Cu at (158.4, 144.5)
- added J1: Conn_02x02_Odd_Even, Connector_PinHeader_2.54mm:PinHeader_2x02_P2.54mm_Vertical, F.Cu at (225.4, 106.4)
- added J13: USB_A_Stacked, Connector_USB:USB_A_Wuerth_61400826021_Horizontal_Stacked, F.Cu at (111.4, 79.8)
- added J14: Conn_01x04, Connector_JST:JST_SH_SM04B-SRSS-TB_1x04-1MP_P1.00mm_Horizontal, F.Cu at (107.3, 114.3)
- added J15: Conn_01x20, Connector_PinHeader_2.54mm:PinHeader_1x20_P2.54mm_Vertical, F.Cu at (111.8, 107.7)
- added J16: Conn_01x04, Connector_PinHeader_2.54mm:PinHeader_1x04_P2.54mm_Vertical, F.Cu at (230.4, 93.8)
- added J17: Barrel_Jack_Switch, Connector_BarrelJack:BarrelJack_Horizontal, F.Cu at (174.0, 120.3)
- added J18: Conn_02x05_Odd_Even, Connector_PinHeader_2.54mm:PinHeader_2x05_P2.54mm_Vertical, F.Cu at (115.6, 81.0)
- added J19: HR871150C, GenericJLCPCB:RJ45_Hanrun_HR871150C_Horizontal, F.Cu at (179.1, 82.9)
- added J3: USB_C_Receptacle_USB2.0_16P, Adafruit:USB_C_Receptacle_HRO_TYPE-C-31-M-31, F.Cu at (203.4, 91.9)
- added JP2: Jumper_2_Open, Connector_PinHeader_2.54mm:PinHeader_1x02_P2.54mm_Vertical, F.Cu at (213.4, 106.4)
- added JP3: Jumper_2_Open, Connector_PinHeader_2.54mm:PinHeader_1x02_P2.54mm_Vertical, F.Cu at (217.9, 106.4)
- added L2: 2.2uH, Inductor_SMD:L_1008_2520Metric, F.Cu at (152.3, 138.4)
- added PORT1: LED_Small, LED_SMD:LED_0603_1608Metric, F.Cu at (105.4, 97.3)
- added PORT2: LED_Small, LED_SMD:LED_0603_1608Metric, F.Cu at (105.4, 99.9)
- added PORT3: LED_Small, LED_SMD:LED_0603_1608Metric, F.Cu at (105.4, 102.5)
- added PORT4: LED_Small, LED_SMD:LED_0603_1608Metric, F.Cu at (105.4, 105.1)
- added R10: 1k, Resistor_SMD:R_0402_1005Metric, F.Cu at (180.2, 42.3)
- added R11: 6.19K, Resistor_SMD:R_0402_1005Metric, F.Cu at (180.2, 44.3)
- added R12: 1k, Resistor_SMD:R_0402_1005Metric, F.Cu at (180.2, 46.3)
- added R13: 1k, Resistor_SMD:R_0402_1005Metric, F.Cu at (180.2, 48.2)
- added R16: 220, Resistor_SMD:R_0402_1005Metric, F.Cu at (101.9, 94.5)
- added R17: 220, Resistor_SMD:R_0402_1005Metric, F.Cu at (101.9, 96.4)
- added R18: 470, Resistor_SMD:R_0402_1005Metric, F.Cu at (101.9, 98.4)
- added R19: 0.1/1% PT2512K 070R1L, Resistor_SMD:R_2512_6332Metric, F.Cu at (128.7, 58.1)
- added R20: 4.7K, Resistor_SMD:R_0402_1005Metric, F.Cu at (119.8, 116.0)
- added R21: 10K, Resistor_SMD:R_0402_1005Metric, F.Cu at (119.8, 118.0)
- added R22: 10K, Resistor_SMD:R_0402_1005Metric, F.Cu at (119.8, 119.9)
- added R23: 10K, Resistor_SMD:R_0402_1005Metric, F.Cu at (119.8, 121.9)
- added R24: 4.7K, Resistor_SMD:R_0402_1005Metric, F.Cu at (132.1, 91.7)
- added R25: 4.7K, Resistor_SMD:R_0402_1005Metric, F.Cu at (141.5, 61.9)
- added R26: 2.2K, Resistor_SMD:R_0402_1005Metric, F.Cu at (163.3, 143.2)
- added R27: 10K, Resistor_SMD:R_0402_1005Metric, F.Cu at (148.4, 132.4)
- added R28: 100K(1%), Resistor_SMD:R_0402_1005Metric, F.Cu at (148.4, 134.4)
- added R29: 22.1K(1%), Resistor_SMD:R_0402_1005Metric, F.Cu at (148.4, 136.4)
- added R30: 5.1K(1%), Resistor_SMD:R_0402_1005Metric, F.Cu at (206.5, 84.6)
- added R31: 5.1K(1%), Resistor_SMD:R_0402_1005Metric, F.Cu at (208.5, 84.6)
- added R32: 1.5k, Resistor_SMD:R_0402_1005Metric, F.Cu at (180.2, 50.2)
- added R33: 1k, Resistor_SMD:R_0402_1005Metric, B.Cu at (183.3, 82.2)
- added R34: 1k, Resistor_SMD:R_0402_1005Metric, B.Cu at (183.3, 84.2)
- added SW1: SW_Push, Button_Switch_SMD:SW_Push_1P1T-MP_NO_Horizontal_Alps_SKRTLAE010, F.Cu at (205.1, 109.3)
- added SW2: SW_Push, Button_Switch_SMD:SW_Push_1P1T-MP_NO_Horizontal_Alps_SKRTLAE010, F.Cu at (205.1, 114.7)
- added U10: TLV62569DBV, Package_TO_SOT_SMD:SOT-23-5, F.Cu at (159.5, 131.8)
- added U4: IPGRI, Package_DFN_QFN:QFN-32-1EP_4x4mm_P0.4mm_EP2.65x2.65mm, F.Cu at (182.3, 65.9)
- added U6: INA219AxD, Package_SO:SOIC-8_3.9x4.9mm_P1.27mm, F.Cu at (143.2, 56.2)
- added U7: CH334F, Package_DFN_QFN:QFN-24-1EP_4x4mm_P0.5mm_EP2.7x2.7mm, F.Cu at (122.5, 87.3)
- added U8: MT9700_SY6280, Package_TO_SOT_SMD:SOT-23-5, F.Cu at (127.9, 111.4)
- added U9: MT9700_SY6280, Package_TO_SOT_SMD:SOT-23-5, F.Cu at (127.9, 116.0)
- added Y2: 25Mhz 12pf, Crystal:Crystal_SMD_3225-4Pin_3.2x2.5mm, F.Cu at (173.8, 66.6)
- added Y3: 12MHz, Crystal:Crystal_SMD_3225-4Pin_3.2x2.5mm, F.Cu at (116.7, 84.4)
- J10, J11, J12, J5, J6, J7: value Conn_01x22 -> Conn_01x20; footprint Connector_PinHeader_2.54mm:PinHeader_1x22_P2.54mm_Vertical -> Connector_PinHeader_2.54mm:PinHeader_1x20_P2.54mm_Vertical
- J2, J4, J9: moved to B.Cu
- moved J4 5.08 mm to (115.6, 74.9), turned to -90 degrees
- moved J9 5.08 mm to (147.3, 122.9), turned to -90 degrees
- moved J2 5.08 mm to (142.2, 74.9), turned to -90 degrees
Connections:
- net /P4/CHIP_PU renamed /RESET
- net /RMII_CLK renamed /P4/GPIO32
- net /RMII_CRSDV renamed /P4/GPIO28
- net /RMII_RXD0 renamed /P4/GPIO29
- net /RMII_RXD1 renamed /P4/GPIO30
- net /RMII_RXER renamed /P4/GPIO31
- net /RMII_TXD0 renamed /P4/GPIO34
- net /RMII_TXEN renamed /P4/GPIO33
- J2 pad 1: Net-(J10-Pin_15) -> Net-(J10-Pin_13)
- J2 pad 2: Net-(J10-Pin_16) -> Net-(J10-Pin_14)
- J2 pad 3: Net-(J10-Pin_17) -> Net-(J10-Pin_15)
- J2 pad 4: Net-(J10-Pin_18) -> Net-(J10-Pin_16)
- J2 pad 5: Net-(J10-Pin_19) -> Net-(J10-Pin_17)
- J2 pad 6: Net-(J10-Pin_20) -> Net-(J10-Pin_18)
- J2 pad 7: Net-(J10-Pin_21) -> Net-(J10-Pin_19)
- J2 pad 8: Net-(J10-Pin_22) -> Net-(J10-Pin_20)
- J5 pad 1: unconnected-(J5-Pin_1-Pad1) -> Net-(J5-Pin_1)
- J5 pad 14: unconnected-(J5-Pin_14-Pad14) -> Net-(J5-Pin_14)
- J5 pad 6: Net-(J5-Pin_6) -> unconnected-(J5-Pin_6-Pad6)
- J5 pad 7: Net-(J5-Pin_7) -> unconnected-(J5-Pin_7-Pad7)
- J9 pad 1: Net-(J5-Pin_7) -> Net-(J5-Pin_14)
- J9 pad 2: Net-(J5-Pin_6) -> Net-(J5-Pin_5)
- J9 pad 3: Net-(J5-Pin_5) -> Net-(J5-Pin_4)
- J9 pad 4: Net-(J5-Pin_4) -> Net-(J5-Pin_3)
- J9 pad 5: Net-(J5-Pin_3) -> Net-(J5-Pin_2)
- J9 pad 6: Net-(J5-Pin_2) -> Net-(J5-Pin_1)
- U2 pad 104: /P4/GPIO0/ADC -> /NEOPIXEL_WAKE
- U2 pad 66: /RMII_TXD1 -> /SDA_BOOT
- U2 pad 68: /RMII_TXER -> /SCL
- U2 pad 81: /P4/GPIO40 -> /Ethernet/RMII_TXEN
- U2 pad 82: /P4/GPIO41 -> /Ethernet/RMII_TXD0
- U2 pad 83: /P4/GPIO42 -> /Ethernet/RMII_TXD1
- U2 pad 86: /P4/GPIO44 -> /Ethernet/RMII_CLK
- U2 pad 87: /P4/GPIO45 -> /Ethernet/RMII_CRSDV
- U2 pad 88: /P4/GPIO46 -> /Ethernet/RMII_RXD0
- U2 pad 89: /P4/GPIO47 -> /Ethernet/RMII_RXD1
Routing:
- net Net-(J10-Pin_15): track 17.3 -> 0.00 mm
- net /P4/FLASH_D: track 0.00 -> 9.24 mm
- net /P4/FLASH_CK: track 0.00 -> 8.05 mm
- net Net-(J10-Pin_18): track 7.15 -> 0.00 mm
- net /P4/FLASH_Q: track 0.00 -> 7.15 mm

Commit message: Fault circuit getting close
Parts:
- added REF**: WS2812B-4020, WorldSemi:WS2812B-4020, F.Cu at (160.0, 64.5)
Changed lines of the file:
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@@
 		)
+	)
+	(footprint "WorldSemi:WS2812B-4020"
+		(layer "F.Cu")
+		(at 160.02 64.47)
+		(property "Reference" "REF**"
+			(at 0 -2.25 0)
+			(unlocked yes)
+			(layer "F.SilkS")
+			(effects
+				(font
+					(size 1 1)
+					(thickness 0.1)
+				)
+			)
+		)
+		(property "Value" "WS2812B-4020"
+			(at 0 1 0)
+			(unlocked yes)
+			(layer "F.Fab")
+			(effects
+				(font
+					(size 1 1)
+					(thickness 0.15)
+				)
+			)
+		)
+		(property "Datasheet" ""
+			(at 0 0 0)
+			(unlocked yes)
+			(layer "F.Fab")
+			(hide yes)
+			(effects
+				(font
+					(size 1 1)
+					(thickness 0.15)
+				)
+			)
+		)
+		(property "Description" ""
+			(at 0 0 0)
+			(unlocked yes)
+			(layer "F.Fab")
+			(hide yes)
+			(effects
+				(font
+					(size 1 1)
+					(thickness 0.15)
+				)
+			)
+		)
+		(attr smd)
+		(duplicate_pad_numbers_are_jumpers no)
+		(fp_text user "${REFERENCE}"
+			(at 0 2.5 0)
+			(unlocked yes)
+			(layer "F.Fab")
+			(effects
+				(font
+					(size 1 1)
+					(thickness 0.15)
+				)
+			)
+		)
+		(pad "1" smd roundrect
+			(at -0.65 0.425)
+			(size 1.3 0.42)
+			(layers "F.Cu" "F.Mask" "F.Paste")
+			(roundrect_rratio 0.15)
+		)
+		(pad "2" smd roundrect
+			(at -0.65 -0.425)
+			(size 1.3 0.42)
+			(layers "F.Cu" "F.Mask" "F.Paste")
+			(roundrect_rratio 0.15)
+		)
+		(pad "3" smd roundrect
+			(at -0.65 -1.275)
+			(size 1.3 0.42)
+			(layers "F.Cu" "F.Mask" "F.Paste")
+			(roundrect_rratio 0.15)
+		)
+		(pad "4" smd roundrect
+			(at -0.65 1.275)
+			(size 1.3 0.42)
+			(layers "F.Cu" "F.Mask" "F.Paste")
+			(roundrect_rratio 0.15)
+		)
+		(embedded_fonts no)
 	)
 	(footprint "Connector_PinHeader_2.54mm:PinHeader_2x02_P2.54mm_Vertical"

Commit message: where I'm at. fault not needed
Parts:
- added D10: BAT54C, Package_TO_SOT_SMD:SOT-23, B.Cu at (133.3, 111.5)
- added D11: BAT54C, Package_TO_SOT_SMD:SOT-23, B.Cu at (138.4, 111.5)
- added D12: BAT54C, Package_TO_SOT_SMD:SOT-23, B.Cu at (143.5, 111.5)
- added D13: BAT54C, Package_TO_SOT_SMD:SOT-23, B.Cu at (148.6, 111.5)
- added D14: BAT54C, Package_TO_SOT_SMD:SOT-23, B.Cu at (153.3, 111.5)
- added D15: BAT54C, Package_TO_SOT_SMD:SOT-23, B.Cu at (158.8, 111.5)
- added D16: BAT54C, Package_TO_SOT_SMD:SOT-23, B.Cu at (113.0, 116.6)
- added D17: BAT54C, Package_TO_SOT_SMD:SOT-23, B.Cu at (138.4, 116.5)
- added D18: BAT54C, Package_TO_SOT_SMD:SOT-23, B.Cu at (118.1, 116.5)
- added D19: BAT54C, Package_TO_SOT_SMD:SOT-23, B.Cu at (143.5, 116.5)
- added D20: BAT54C, Package_TO_SOT_SMD:SOT-23, B.Cu at (123.2, 116.5)
- added D21: BAT54C, Package_TO_SOT_SMD:SOT-23, B.Cu at (148.6, 116.5)
- added D22: BAT54C, Package_TO_SOT_SMD:SOT-23, B.Cu at (128.3, 116.5)
- added D23: BAT54C, Package_TO_SOT_SMD:SOT-23, B.Cu at (153.7, 116.5)
- added D24: BAT54C, Package_TO_SOT_SMD:SOT-23, B.Cu at (133.3, 116.5)
- added D25: BAT54C, Package_TO_SOT_SMD:SOT-23, B.Cu at (158.8, 116.5)
- added D5: BAT54C, Package_TO_SOT_SMD:SOT-23, B.Cu at (113.0, 111.5)
- added D6: BAT54C, Package_TO_SOT_SMD:SOT-23, B.Cu at (118.1, 111.5)
- added D7: BAT54C, Package_TO_SOT_SMD:SOT-23, B.Cu at (123.2, 111.5)
- added D9: BAT54C, Package_TO_SOT_SMD:SOT-23, B.Cu at (128.3, 111.5)
- added U5: TLV7031DBV, Package_TO_SOT_SMD:SOT-23-5, F.Cu at (173.3, 139.3)
- D1: footprint LED_SMD:LED_WS2812B_PLCC4_5.0x5.0mm_P3.2mm -> WorldSemi:WS2812B-4020
Connections:
- net /USB Host/POWER_ON renamed /FaultCheck/ENABLE_OUT
- net Net-(J10-Pin_1) renamed /DeviceUnderTest/T1
- net Net-(J10-Pin_10) renamed /DeviceUnderTest/T10
- net Net-(J10-Pin_11) renamed /DeviceUnderTest/ARDUINO_IOREF
- net Net-(J10-Pin_12) renamed /DeviceUnderTest/ARDUINO_RESET
- net Net-(J10-Pin_13) renamed /DeviceUnderTest/T13
- net Net-(J10-Pin_14) renamed /DeviceUnderTest/T14
- net Net-(J10-Pin_15) renamed /DeviceUnderTest/T15
- net Net-(J10-Pin_16) renamed /DeviceUnderTest/T16
- net Net-(J10-Pin_17) renamed /DeviceUnderTest/T17
- net Net-(J10-Pin_18) renamed /DeviceUnderTest/T18
- net Net-(J10-Pin_19) renamed /DeviceUnderTest/T19
- net Net-(J10-Pin_2) renamed /DeviceUnderTest/T2
- net Net-(J10-Pin_20) renamed /DeviceUnderTest/T20
- net Net-(J10-Pin_3) renamed /DeviceUnderTest/T3
- net Net-(J10-Pin_4) renamed /DeviceUnderTest/T4
- net Net-(J10-Pin_5) renamed /DeviceUnderTest/T5
- net Net-(J10-Pin_6) renamed /DeviceUnderTest/T6
- net Net-(J10-Pin_7) renamed /DeviceUnderTest/T7
- net Net-(J10-Pin_8) renamed /DeviceUnderTest/T8
- net Net-(J10-Pin_9) renamed /DeviceUnderTest/T9
- net Net-(J5-Pin_1) renamed /DeviceUnderTest/B1
- net Net-(J5-Pin_14) renamed /DeviceUnderTest/B14
- net Net-(J5-Pin_2) renamed /DeviceUnderTest/B2
- net Net-(J5-Pin_3) renamed /DeviceUnderTest/B3
- net Net-(J5-Pin_4) renamed /DeviceUnderTest/B4
- net Net-(J5-Pin_5) renamed /DeviceUnderTest/B5
- C50 pad 1: unconnected-(C50-Pad1) -> /USB Host/SWITCHED_3V3
- C50 pad 2: unconnected-(C50-Pad2) -> GND
- J5 pad 10: unconnected-(J5-Pin_10-Pad10) -> /DeviceUnderTest/B10
- J5 pad 11: unconnected-(J5-Pin_11-Pad11) -> /DeviceUnderTest/B11
- J5 pad 12: unconnected-(J5-Pin_12-Pad12) -> /DeviceUnderTest/B12
- J5 pad 13: unconnected-(J5-Pin_13-Pad13) -> /DeviceUnderTest/B13
- J5 pad 15: unconnected-(J5-Pin_15-Pad15) -> /DeviceUnderTest/B15
- J5 pad 16: unconnected-(J5-Pin_16-Pad16) -> /DeviceUnderTest/B16
- J5 pad 17: unconnected-(J5-Pin_17-Pad17) -> /DeviceUnderTest/B17
- J5 pad 18: unconnected-(J5-Pin_18-Pad18) -> /DeviceUnderTest/B18
- J5 pad 19: unconnected-(J5-Pin_19-Pad19) -> /DeviceUnderTest/B19
- J5 pad 20: unconnected-(J5-Pin_20-Pad20) -> /DeviceUnderTest/B20
- J5 pad 6: unconnected-(J5-Pin_6-Pad6) -> /DeviceUnderTest/B6
- J5 pad 7: unconnected-(J5-Pin_7-Pad7) -> /DeviceUnderTest/B7
- J5 pad 8: unconnected-(J5-Pin_8-Pad8) -> /DeviceUnderTest/B8
- J5 pad 9: unconnected-(J5-Pin_9-Pad9) -> /DeviceUnderTest/B9

Commit message: Remove fault stuff
Parts:
- removed D10, D11, D12, D13, D14, D15, D16, D17, D18, D19, D20, D21, D22, D23, D24, D25, D5, D6, D7, D9: BAT54C, Package_TO_SOT_SMD:SOT-23
- removed REF**: WS2812B-4020, WorldSemi:WS2812B-4020
- removed U5: TLV7031DBV, Package_TO_SOT_SMD:SOT-23-5
- added J8: Conn_01x02, Connector_PinHeader_2.54mm:PinHeader_1x02_P2.54mm_Vertical, F.Cu at (99.6, 164.9)
- added R100: 2.2K, Resistor_SMD:R_0402_1005Metric, F.Cu at (116.2, 155.6)
- added R101: 2.2K, Resistor_SMD:R_0402_1005Metric, F.Cu at (116.2, 157.6)
- added R102: 2.2K, Resistor_SMD:R_0402_1005Metric, F.Cu at (116.2, 159.6)
- added R103: 2.2K, Resistor_SMD:R_0402_1005Metric, F.Cu at (116.2, 161.6)
- added R104: 2.2K, Resistor_SMD:R_0402_1005Metric, F.Cu at (137.2, 117.8)
- added R105: 2.2K, Resistor_SMD:R_0402_1005Metric, F.Cu at (119.1, 145.7)
- added R106: 2.2K, Resistor_SMD:R_0402_1005Metric, F.Cu at (119.1, 147.7)
- added R107: 2.2K, Resistor_SMD:R_0402_1005Metric, F.Cu at (119.1, 149.7)
- added R108: 2.2K, Resistor_SMD:R_0402_1005Metric, F.Cu at (119.1, 151.7)
- added R109: 2.2K, Resistor_SMD:R_0402_1005Metric, F.Cu at (119.1, 153.7)
- added R110: 2.2K, Resistor_SMD:R_0402_1005Metric, F.Cu at (119.1, 155.6)
- added R111: 2.2K, Resistor_SMD:R_0402_1005Metric, F.Cu at (119.1, 157.6)
- added R112: 2.2K, Resistor_SMD:R_0402_1005Metric, F.Cu at (119.1, 159.6)
- added R113: 2.2K, Resistor_SMD:R_0402_1005Metric, F.Cu at (119.1, 161.6)
- added R14: R_Protect, Resistor_SMD:R_0402_1005Metric, F.Cu at (98.7, 147.7)
- added R15: R_Protect, Resistor_SMD:R_0402_1005Metric, F.Cu at (98.7, 149.7)
- added R35: R_Protect, Resistor_SMD:R_0402_1005Metric, F.Cu at (98.7, 151.7)
- added R36: R_Protect, Resistor_SMD:R_0402_1005Metric, F.Cu at (98.7, 153.7)
- added R37: R_Protect, Resistor_SMD:R_0402_1005Metric, F.Cu at (98.7, 155.6)
- added R38: R_Protect, Resistor_SMD:R_0402_1005Metric, F.Cu at (98.7, 157.6)
- added R39: R_Protect, Resistor_SMD:R_0402_1005Metric, F.Cu at (98.7, 159.6)
- added R40: R_Protect, Resistor_SMD:R_0402_1005Metric, F.Cu at (98.7, 161.6)
- added R41: R_Protect, Resistor_SMD:R_0402_1005Metric, F.Cu at (137.2, 92.4)
- added R42: R_Protect, Resistor_SMD:R_0402_1005Metric, F.Cu at (101.7, 145.7)
- added R43: R_Protect, Resistor_SMD:R_0402_1005Metric, F.Cu at (101.7, 147.7)
- added R44: R_Protect, Resistor_SMD:R_0402_1005Metric, F.Cu at (101.7, 149.7)
- added R45: R_Protect, Resistor_SMD:R_0402_1005Metric, F.Cu at (101.7, 151.7)
- added R46: R_Protect, Resistor_SMD:R_0402_1005Metric, F.Cu at (101.7, 153.7)
- added R47: R_Protect, Resistor_SMD:R_0402_1005Metric, F.Cu at (101.7, 155.6)
- added R48: R_Protect, Resistor_SMD:R_0402_1005Metric, F.Cu at (101.7, 157.6)
- added R49: R_Protect, Resistor_SMD:R_0402_1005Metric, F.Cu at (101.7, 159.6)
- added R50: R_Protect, Resistor_SMD:R_0402_1005Metric, F.Cu at (101.7, 161.6)
- added R51: R_Protect, Resistor_SMD:R_0402_1005Metric, F.Cu at (104.6, 143.7)
- added R52: R_Protect, Resistor_SMD:R_0402_1005Metric, F.Cu at (104.6, 145.7)
- added R53: R_Protect, Resistor_SMD:R_0402_1005Metric, F.Cu at (104.6, 147.7)
- added R54: R_Protect, Resistor_SMD:R_0402_1005Metric, F.Cu at (104.6, 149.7)
- added R55: R_Protect, Resistor_SMD:R_0402_1005Metric, F.Cu at (104.6, 151.7)
- added R56: R_Protect, Resistor_SMD:R_0402_1005Metric, F.Cu at (104.6, 153.7)
- added R57: R_Protect, Resistor_SMD:R_0402_1005Metric, F.Cu at (104.6, 155.6)
- added R58: R_Protect, Resistor_SMD:R_0402_1005Metric, F.Cu at (104.6, 157.6)
- added R59: R_Protect, Resistor_SMD:R_0402_1005Metric, F.Cu at (104.6, 159.6)
- added R60: R_Protect, Resistor_SMD:R_0402_1005Metric, F.Cu at (104.6, 161.6)
- added R61: R_Protect, Resistor_SMD:R_0402_1005Metric, F.Cu at (137.2, 116.5)
- added R62: R_Protect, Resistor_SMD:R_0402_1005Metric, F.Cu at (107.5, 145.7)
- added R63: R_Protect, Resistor_SMD:R_0402_1005Metric, F.Cu at (107.5, 147.7)
- added R64: R_Protect, Resistor_SMD:R_0402_1005Metric, F.Cu at (107.5, 149.7)
- added R65: R_Protect, Resistor_SMD:R_0402_1005Metric, F.Cu at (107.5, 151.7)
- added R66: R_Protect, Resistor_SMD:R_0402_1005Metric, F.Cu at (107.5, 153.7)
- added R67: R_Protect, Resistor_SMD:R_0402_1005Metric, F.Cu at (107.5, 155.6)
- added R68: R_Protect, Resistor_SMD:R_0402_1005Metric, F.Cu at (107.5, 157.6)
- added R69: R_Protect, Resistor_SMD:R_0402_1005Metric, F.Cu at (107.5, 159.6)
- added R70: R_Protect, Resistor_SMD:R_0402_1005Metric, F.Cu at (107.5, 161.6)
- added R74: 2.2K, Resistor_SMD:R_0402_1005Metric, F.Cu at (110.4, 143.7)
- added R75: 2.2K, Resistor_SMD:R_0402_1005Metric, F.Cu at (110.4, 145.7)
- added R76: 2.2K, Resistor_SMD:R_0402_1005Metric, F.Cu at (110.4, 147.7)
- added R77: 2.2K, Resistor_SMD:R_0402_1005Metric, F.Cu at (110.4, 149.7)
- added R78: 2.2K, Resistor_SMD:R_0402_1005Metric, F.Cu at (110.4, 151.7)
- added R79: 2.2K, Resistor_SMD:R_0402_1005Metric, F.Cu at (110.4, 153.7)
- added R8: R_Protect, Resistor_SMD:R_0402_1005Metric, F.Cu at (98.7, 143.7)
- added R80: 2.2K, Resistor_SMD:R_0402_1005Metric, F.Cu at (110.4, 155.6)
- added R81: 2.2K, Resistor_SMD:R_0402_1005Metric, F.Cu at (110.4, 157.6)
- added R82: 2.2K, Resistor_SMD:R_0402_1005Metric, F.Cu at (110.4, 159.6)
- added R83: 2.2K, Resistor_SMD:R_0402_1005Metric, F.Cu at (110.4, 161.6)
- added R84: 2.2K, Resistor_SMD:R_0402_1005Metric, F.Cu at (113.3, 143.7)
- added R85: 2.2K, Resistor_SMD:R_0402_1005Metric, F.Cu at (113.3, 145.7)
- added R86: 2.2K, Resistor_SMD:R_0402_1005Metric, F.Cu at (113.3, 147.7)
- added R87: 2.2K, Resistor_SMD:R_0402_1005Metric, F.Cu at (113.3, 149.7)
- added R88: 2.2K, Resistor_SMD:R_0402_1005Metric, F.Cu at (113.3, 151.7)
- added R89: 2.2K, Resistor_SMD:R_0402_1005Metric, F.Cu at (113.3, 153.7)
- added R9: R_Protect, Resistor_SMD:R_0402_1005Metric, F.Cu at (98.7, 145.7)
- added R90: 2.2K, Resistor_SMD:R_0402_1005Metric, F.Cu at (113.3, 155.6)
- added R91: 2.2K, Resistor_SMD:R_0402_1005Metric, F.Cu at (113.3, 157.6)
- added R92: 2.2K, Resistor_SMD:R_0402_1005Metric, F.Cu at (113.3, 159.6)
- added R93: 2.2K, Resistor_SMD:R_0402_1005Metric, F.Cu at (113.3, 161.6)
- added R94: 2.2K, Resistor_SMD:R_0402_1005Metric, F.Cu at (116.2, 143.7)
- added R95: 2.2K, Resistor_SMD:R_0402_1005Metric, F.Cu at (116.2, 145.7)
- added R96: 2.2K, Resistor_SMD:R_0402_1005Metric, F.Cu at (116.2, 147.7)
- added R97: 2.2K, Resistor_SMD:R_0402_1005Metric, F.Cu at (116.2, 149.7)
- added R98: 2.2K, Resistor_SMD:R_0402_1005Metric, F.Cu at (116.2, 151.7)
- added R99: 2.2K, Resistor_SMD:R_0402_1005Metric, F.Cu at (116.2, 153.7)
- moved C49 75.2 mm to (88.0, 123.2)
- moved R19 75.2 mm to (81.3, 116.5)
- moved R25 75.2 mm to (94.1, 120.3)
- moved U6 75.2 mm to (95.7, 114.6)
- moved J3 22.9 mm to (181.6, 98.8)
- moved C46 10.9 mm to (127.0, 90.8)
- moved C47 10.7 mm to (127.0, 92.4)
- moved C48 7.59 mm to (127.0, 89.5)
- moved Y3 6.53 mm to (123.2, 84.8)
- moved U7 2.52 mm to (122.5, 89.9), turned to -90 degrees
Connections:
- net /FaultCheck/ENABLE_OUT renamed /USB Host/POWER_ON
Routing:
- added copper zone on B.Cu, net GND
- added copper zone on F.Cu, net GND
- added copper zone on In1.Cu, net GND
