File: ethernet.kicad_sch (KiCad schematic)
At the start: 18 parts, among them J1 HR871150C, U4 IPGRI, Y2 25Mhz

Commit message: Getting close. Fault circuit left
Parts:
- removed C44: 100nF, symbol Device:C_Small
- removed J1: HR871150C, Connector_RJ:RJ45_Abracon_ARJP11A-MA_Horizontal, symbol Connector:RJ45_Abracon_ARJP11A-MASA-B-A-EMU2
- removed U5: (no value), symbol PoE-Module:SIL-Module
- added J19: HR871150C, GenericJLCPCB:RJ45_Hanrun_HR871150C_Horizontal, symbol GenericJLC:RJ45_10_100_PoE_LED
- added R32: 1.5k, Resistor_SMD:R_0402_1005Metric, symbol Device:R_Small
- added R33, R34: 1k, Resistor_SMD:R_0402_1005Metric, symbol Device:R_Small
- C35, C38, C40, C43: footprint (none) -> Capacitor_SMD:C_0402_1005Metric
- C36, C37, C39: footprint (none) -> Capacitor_SMD:C_0603_1608Metric
- C41: value 100nF -> 18pF; footprint (none) -> Capacitor_SMD:C_0402_1005Metric
- C42: value TODO -> 18pF; footprint (none) -> Capacitor_SMD:C_0402_1005Metric
- R10, R12, R13: value R_Pull -> 1k; footprint (none) -> Resistor_SMD:R_0402_1005Metric
- R11: footprint (none) -> Resistor_SMD:R_0402_1005Metric
- Y2: value 25Mhz -> 25Mhz 12pf; footprint (none) -> Crystal:Crystal_SMD_3225-4Pin_3.2x2.5mm
Connections:
- net +3.3V: now also J19.11, R32.1
- net GND: now also J19.SH, R34.2
- net MDC: now also R32.2
- net RN: now also J19.5 (RD-)
- net RP: now also J19.4 (RD+)
- net TN: now also J19.2 (TD-)
- net TP: now also J19.1 (TD+)
- net LED_100MB_ACT renamed LED3
- net LED3: now also J19.13
- net LED_LINK renamed LED0
- net LED0: now also R33.2
- net TCT renamed CT
- net CT: now also J19.3 (CT)
- new net: J19.12, R33.1
- new net: J19.14, R34.1
- new net POWER1: J19.10 (Vc4)
- new net POWER2: J19.9 (Vc3)
- no-connect marks 5 -> 7
Other:
- removed sheet EthernetPoEDiode
- note added: "No real Mode A PoE."

Commit message: more routing
Parts:
- added R50: 1.5k, Resistor_SMD:R_0402_1005Metric, symbol Device:R_Small
- R32: now not fitted
Connections:
- net +3.3V: now also R50.1
- net MDIO: now also R50.2
Changed lines of the file:
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@@
 		(color 0 0 0 0)
 	)
+	(junction
+		(at 134.62 73.66)
+		(diameter 0)
+		(color 0 0 0 0)
+	)
 	(no_connect
 		(at 135.89 105.41)
@@
 	(wire
 		(pts
+			(xy 124.46 73.66) (xy 134.62 73.66)
+		)
+		(stroke
+			(width 0)
+			(type default)
+		)
+	)
+	(wire
+		(pts
 			(xy 226.06 109.22) (xy 217.17 109.22)
 		)
@@
 		)
 	)
+	(wire
+		(pts
+			(xy 134.62 73.66) (xy 135.89 73.66)
+		)
+		(stroke
+			(width 0)
+			(type default)
+		)
+	)
 	(label "25M_XI"
 		(at 215.9 139.7 0)
@@
 	(hierarchical_label "MDIO"
 		(shape input)
-		(at 135.89 73.66 180)
+		(at 124.46 73.66 180)
 		(effects
 			(font
@@
 	)
 	(symbol
+		(lib_id "Device:R_Small")
+		(at 134.62 71.12 0)
+		(unit 1)
+		(body_style 1)
+		(exclude_from_sim no)
+		(in_bom yes)
+		(on_board yes)
+		(in_pos_files yes)
+		(dnp no)
+		(property "Reference" "R50"
+			(at 135.89 66.548 0)
+			(show_name no)
+			(do_not_autoplace no)
+			(effects
+				(font
+					(size 1.016 1.016)
+				)
+				(justify left)
+			)
+		)
+		(property "Value" "1.5k"
+			(at 135.636 64.77 0)
+			(show_name no)
+			(do_not_autoplace no)
+			(effects
+				(font
+					(size 1.27 1.27)
+				)
+				(justify left)
+			)
+		)
+		(property "Footprint" "Resistor_SMD:R_0402_1005Metric"
+			(at 134.62 71.12 0)
+			(hide yes)
+			(show_name no)
+			(do_not_autoplace no)
+			(effects
+				(font
+					(size 1.27 1.27)
+				)
+			)
+		)
+		(property "Datasheet" ""
+			(at 134.62 71.12 0)
+			(hide yes)
+			(show_name no)
+			(do_not_autoplace no)
+			(effects
+				(font
+					(size 1.27 1.27)
+				)
+			)
+		)
+		(property "Description" "Resistor, small symbol"
+			(at 134.62 71.12 0)
+			(hide yes)
+			(show_name no)
+			(do_not_autoplace no)
+			(effects
+				(font
+					(size 1.27 1.27)
+				)
+			)
+		)
+		(pin "1"
+		)
+		(pin "2"
+		)
+		(instances
+			(project "p4hil"
+				(path "/b29b188c-1e37-42da-9ef2-78e9f87e21db/16022e0a-5f3f-4f99-9755-d71b2286f4b7"
+					(reference "R50")
+					(unit 1)
+				)
+			)
+		)
+	)
+	(symbol
 		(lib_id "Device:C_Small")
 		(at 215.9 144.78 0)
@@
 		(on_board yes)
 		(in_pos_files yes)
-		(dnp no)
+		(dnp yes)
 		(property "Reference" "R32"
-			(at 133.35 67.3099 0)
+			(at 126.238 65.278 0)
 			(show_name no)
 			(do_not_autoplace no)
@@
 		)
 		(property "Value" "1.5k"
-			(at 123.444 67.31 0)
+			(at 125.222 67.056 0)
 			(show_name no)
 			(do_not_autoplace no)
@@
 					(unit 1)
 				)
+			)
+		)
+	)
+	(symbol
+		(lib_id "power:+3.3V")
+		(at 134.62 68.58 0)
+		(unit 1)
+		(body_style 1)
+		(exclude_from_sim no)
+		(in_bom yes)
+		(on_board yes)
+		(in_pos_files yes)
+		(dnp no)
+		(fields_autoplaced yes)
+		(property "Reference" "#PWR061"
+			(at 134.62 72.39 0)
+			(hide yes)
+			(show_name no)
+			(do_not_autoplace no)
+			(effects
+				(font
+					(size 1.27 1.27)
+				)
+			)
+		)
+		(property "Value" "+3.3V"
+			(at 134.62 63.5 0)
+			(show_name no)
+			(do_not_autoplace no)
+			(effects
+				(font
+					(size 1.27 1.27)
+				)
+			)
+		)
+		(property "Footprint" ""
+			(at 134.62 68.58 0)
+			(hide yes)
+			(show_name no)
+			(do_not_autoplace no)
+			(effects
+				(font
+					(size 1.27 1.27)
+				)
+			)
+		)
+		(property "Datasheet" ""
+			(at 134.62 68.58 0)
+			(hide yes)
+			(show_name no)
+			(do_not_autoplace no)
+			(effects
+				(font
+					(size 1.27 1.27)
+				)
+			)
+		)
+		(property "Description" "Power symbol creates a global label with name \"+3.3V\""
+			(at 134.62 68.58 0)
+			(hide yes)
+			(show_name no)
+			(do_not_autoplace no)
+			(effects
+				(font
+					(size 1.27 1.27)
+				)
+			)
+		)
+		(pin "1"
+		)
+		(instances
+			(project "p4hil"
+				(path "/b29b188c-1e37-42da-9ef2-78e9f87e21db/16022e0a-5f3f-4f99-9755-d71b2286f4b7"
+					(reference "#PWR061")
+					(unit 1)
+				)

Commit message: Add IO expanders, swap ethernet and move USB LEDs
Parts:
- removed J19: HR871150C, GenericJLCPCB:RJ45_Hanrun_HR871150C_Horizontal, symbol GenericJLC:RJ45_10_100_PoE_LED
- added C44: 100nF, Capacitor_SMD:C_0402_1005Metric, symbol Device:C_Small
- added J19: RJ45_Hanrun_HR911105A_Horizontal, Connector_RJ:RJ45_Hanrun_HR911105A_Horizontal, symbol Connector:RJ45_Hanrun_HR911105A_Horizontal
Connections:
- net +3.3V: now also J19.9
- net GND: now also C44.2, J19.8, J19.SH
- net LED3: now also J19.12
- net RN: now also J19.6 (RD-)
- net RP: now also J19.3 (RD+)
- net TN: now also J19.2 (TD-)
- net TP: now also J19.1 (TD+)
- net at R33.1: now also J19.10
- net at R34.1: now also J19.11
- net CT renamed TCT
- net TCT: now also J19.4 (TCT)
- new net RCT: C44.1, J19.5 (RCT)
- no-connect marks 7 -> 5
Other:
- note removed: "No real Mode A PoE."
- moved on the sheet: R33, R34
